Commit message: update lidar

File: src/sjtu_drone/sjtu_drone_description/urdf/sjtu_drone.urdf.xacro (robot description, xacro)
@@ -42,4 +42,11 @@
   </joint>
   <link name="sonar_link"/>
+  <!-- 2-D LiDAR — mounted on top of the drone body -->
+  <joint name="lidar_joint" type="fixed">
+    <parent link="base_link" />
+    <child link="lidar_link" />
+    <origin rpy="0 0 0" xyz="0 0 0.1"/>
+  </joint>
+  <link name="lidar_link"/>
   <joint name="front_cam_joint" type="fixed">
     <origin rpy="0 0 0" xyz="0.2 0 0"/>
@@ -203,4 +210,39 @@
     </sensor>
   </gazebo>
+  <!-- 2-D LiDAR (360° horizontal scan) -->
+  <gazebo reference="lidar_link">
+    <sensor name="lidar" type="gpu_lidar">
+      <always_on>true</always_on>
+      <visualize>true</visualize>
+      <update_rate>10</update_rate>
+      <lidar>
+        <scan>
+          <horizontal>
+            <samples>360</samples>
+            <resolution>1</resolution>
+            <min_angle>-3.14159265</min_angle>
+            <max_angle>3.14159265</max_angle>
+          </horizontal>
+          <vertical>
+            <samples>1</samples>
+            <resolution>1</resolution>
+            <min_angle>0</min_angle>
+            <max_angle>0</max_angle>
+          </vertical>
+        </scan>
+        <range>
+          <min>0.1</min>
+          <max>30.0</max>
+          <resolution>0.01</resolution>
+        </range>
+        <noise>
+          <type>gaussian</type>
+          <mean>0</mean>
+          <stddev>0.01</stddev>
+        </noise>
+      </lidar>
+      <gz_frame_id>laser</gz_frame_id>
+    </sensor>
+  </gazebo>
   <!-- Contact sensor -->
   <gazebo reference="base_link">

Commit message: Update launch and configuration files for maze world; adjust spawn positions and add IMU support

File: src/sjtu_drone/sjtu_drone_description/urdf/sjtu_drone.urdf.xacro (robot description, xacro)
@@ -42,4 +42,10 @@
   </joint>
   <link name="sonar_link"/>
+  <joint name="imu_joint" type="fixed">
+    <parent link="base_link" />
+    <child link="imu_link" />
+    <origin rpy="0 0 0" xyz="0 0 0"/>
+  </joint>
+  <link name="imu_link"/>
   <!-- 2-D LiDAR — mounted on top of the drone body -->
   <joint name="lidar_joint" type="fixed">
@@ -97,5 +103,5 @@
   <!-- Sensors (gz-sim native, no Classic plugin children) -->
   <!-- IMU sensor -->
-  <gazebo reference="base_link">
+  <gazebo reference="imu_link">
     <sensor name='sensor_imu' type='imu'>
       <always_on>true</always_on>
@@ -113,5 +119,5 @@
         </linear_acceleration>
       </imu>
-      <gz_frame_id>${mp['namespace']}/base_link</gz_frame_id>
+      <gz_frame_id>${mp['namespace']}/imu_link</gz_frame_id>
     </sensor>
   </gazebo>
